File: kicad/lin2sw.kicad_pcb (KiCad board)
At the start: 2 copper layers, 27 x 13 mm, 20 parts, among them P1 TO220, U1 LM2675-5.0

Commit message: minor mods to layout. Gerbers ready for fab
Parts:
- moved REF** 0.20 mm to (50.3, 32.8)
- moved REF** 0.20 mm to (48.7, 32.8)
Other:
- net class 0.5 added: clearance 0.2, trace_width 0.5, via_dia 0.8, via_drill 0.4
